File: PCB/splitkeybaord.kicad_pcb (KiCad board)
At the start: 2 copper layers, 335.6 x 98 mm, 249 parts, among them J3 TFTTT, J4 TFTTT, J5 BATT, J6 BATT, J7 NFC2, J8 NFC2, Q1 AO3400A, Q2 AO3400A, SW1 SW_Push, SW10 SW_Push, SW11 SW_Push, SW12 SW_Push, SW13 SW_Push, SW14 SW_Push, SW15 SW_Push, SW16 SW_Push, SW17 SW_Push, SW18 SW_Push, SW19 SW_Push, SW2 SW_Push, SW20 SW_Push, SW21 SW_Push, SW22 SW_Push, SW23 SW_Push, SW24 SW_Push, SW25 SW_Push, SW26 SW_Push, SW27 SW_Push, SW28 SW_Push, SW29 SW_Push, SW3 SW_Push, SW30 SW_Push, SW31 SW_Push, SW32 SW_Push, SW33 SW_Push, SW34 SW_Push, SW35 SW_Push, SW36 SW_Push, SW37 SW_Push, SW38 SW_Push, SW39 SW_Push, SW4 SW_Push, SW40 SW_Push, SW41 SW_Push, SW42 SW_Push, SW43 RotaryEncoder_Switch, SW44 RotaryEncoder_Switch, SW47 reset, SW48 boot, SW49 reset, SW5 SW_Push, SW50 boot, SW51 SW_Wuerth_450301014042, SW52 SW_Wuerth_450301014042, SW6 SW_Push, SW7 SW_Push, SW8 SW_Push, SW9 SW_Push, U1 ESP32-S3-WROOM-1-N4R8, U2 ESP32-S3-WROOM-1-N4R8, U3 TP4056_C725790, U4 TP4056_C725790, U5 ME6211A33M3G-N, U6 ME6211A33M3G-N

Commit message: minorupdates
Parts:
- added mouse-bite-5mm-slot: VAL**, Panelization:mouse-bite-5mm-slot, F.Cu at (45.7, 8.47)
- added mouse-bite-5mm-slot: VAL**, Panelization:mouse-bite-5mm-slot, F.Cu at (288.6, 8.45)
Routing:
- net /left/COL5: track 92.7 -> 107.9 mm
Other:
- board size 335.6 x 98 mm -> 335.7 x 101 mm
